File: kicad/ta191.kicad_pcb (KiCad board)
At the start: 2 copper layers, 83.8 x 64.8 mm, 74 parts, among them J1 PHONO, J2 MC/MM IN, J3 MM OUT, J4 OUTPUT, J5 POWER, J6 ~{MC}, J8 +12V, K1 SRD-S-112D, K2 SRD-S-112D, K51 SRD-S-112D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

Commit message: fix mounting holes
Parts:
- moved H2 1.27 mm to (104.1, 38.1)
Routing:
- net GND: track 251.6 -> 252.7 mm
Changed lines of the file:
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@@
 	(footprint "MountingHole:MountingHole_3.2mm_M3_DIN965_Pad"
 		(layer "F.Cu")
-		(at 105.41 38.1)
+		(at 104.14 38.1)
 		(descr "Mounting Hole 3.2mm, M3, DIN965")
 		(tags "mounting hole 3.2mm m3 din965")
@@
 	)
 	(segment
-		(start 107.95 35.56)
-		(end 105.41 38.1)
+		(start 107.95 41.91)
+		(end 104.14 38.1)
 		(width 1.27)
 		(layer "F.Cu")
@@
 	)
 	(segment
-		(start 107.95 40.64)
-		(end 105.41 38.1)
-		(width 1.27)
-		(layer "F.Cu")
-		(net 1)
-	)
-	(segment
 		(start 53.59 47.24)
 		(end 52.705 46.355)
@@
 	)
 	(segment
-		(start 53.59 55.495)
-		(end 53.59 47.24)
+		(start 107.95 43.18)
+		(end 107.95 41.91)
 		(width 1.27)
 		(layer "F.Cu")
@@
 	)
 	(segment
-		(start 107.95 43.18)
-		(end 107.95 40.64)
+		(start 53.59 55.495)
+		(end 53.59 47.24)
 		(width 1.27)
 		(layer "F.Cu")
@@
 	)
 	(segment
+		(start 107.95 34.29)
+		(end 104.14 38.1)
+		(width 1.27)
+		(layer "F.Cu")
+		(net 1)
+	)
+	(segment
 		(start 55.88 43.18)
 		(end 52.705 46.355)
@@
 	)
 	(segment
+		(start 107.95 33.02)
+		(end 107.95 34.29)
+		(width 1.27)
+		(layer "F.Cu")
+		(net 1)
+	)
+	(segment
 		(start 55.245 30.48)
 		(end 67.31 30.48)
@@
 	)
 	(segment
-		(start 107.95 33.02)
-		(end 107.95 35.56)
-		(width 1.27)
-		(layer "F.Cu")
-		(net 1)
-	)
-	(segment
 		(start 54.61 39.37)
 		(end 54.61 31.115)
@@
 	)
 	(segment
-		(start 91.26 41.545)
-		(end 90.895 41.91)
-		(width 1.27)
-		(layer "B.Cu")
-		(net 19)
-	)
-	(segment
-		(start 103.14 41.545)
-		(end 91.26 41.545)
+		(start 95.52 41.545)
+		(end 97.155 43.18)
 		(width 1.27)
 		(layer "B.Cu")
@@
 	)
 	(segment
+		(start 90.895 41.91)
+		(end 91.26 41.545)
+		(width 1.27)
+		(layer "B.Cu")
+		(net 19)
+	)
+	(segment
 		(start 32.547189 43.18)
 		(end 36.83 43.18)
@@
 	)
 	(segment
-		(start 104.775 43.18)
-		(end 103.14 41.545)
+		(start 91.26 41.545)
+		(end 95.52 41.545)
+		(width 1.27)
+		(layer "B.Cu")
+		(net 19)
+	)
+	(segment
+		(start 97.155 43.18)
+		(end 104.775 43.18)
 		(width 1.27)
 		(layer "B.Cu")
